Commit message: removed rope behavior on sail. Now sail angle is set by a revolution joint (like a servo motor)

File: src/usv_sim/xacro/sailboat_2.xacro (robot description, xacro)
@@ -66,5 +66,5 @@
         <dynamics damping="1.0"/>
         <axis xyz="0 0 1"/>
-        <limit effort="0" velocity="5" lower="-${PI/2}" upper="${PI/2}" />
+        <limit effort="5000000000" velocity="5" lower="-${PI/2}" upper="${PI/2}" />
     </joint>
     <!-- Plugin list -->
